File: hw/logic.kicad_sch (KiCad schematic)
At the start: 39 parts, among them J6 UART, J7 ESP_PWR, SW2 SW_Push, SW3 SW_Push, U7 BMP280, U8 LSM303C, U9 ESP32-C6-MINI-1/U, Y1 32.768k

Commit message: USB fix and schematic cleanup (April work)
Add CR2 ESDA25P35 on the USB lines and tie VBUS straight to +5V, drop
the ESP_PWR header J7, JP9 and the VBAT_MON divider, add R25 4.7k and
wire the LSM303C I2C, remove the external LED output (D9, J4, C18).
Parts:
- removed J7: ESP_PWR, Connector_JST:JST_ZH_B6B-ZR_1x06_P1.50mm_Vertical, symbol Connector:Conn_01x06_Socket
- removed JP9: SolderJumper_2_Open, Jumper:SolderJumper-2_P1.3mm_Open_TrianglePad1.0x1.5mm, symbol Jumper:SolderJumper_2_Open
- added R25, R26: 4.7k, Resistor_SMD:R_0603_1608Metric, symbol Device:R
Connections:
- net +3V3: now also R25.2, R26.2
- net ESP_SCL: now also R25.1
- net ESP_SDA: now also R26.1
- no-connect marks 10 -> 11
